Commit message: fix modelling issues

File: src/chromapi/model/urdf/robot.urdf (robot description, URDF)
Before this commit: robot chromapi, 19 links, 18 joints
Links:
- link chassis_assembly: mass 312.693 -> 1.00501
- link left_coxa_assembly: mass 55.0475 -> 0.102452
- link left_coxa_assembly_2: mass 55.0475 -> 0.102452
- link left_femur_assembly: mass 55.0477 -> 0.10275
- link left_femur_assembly_2: mass 55.0477 -> 0.10275
- link right_coxa_assembly: mass 55.0475 -> 0.102452
- link right_coxa_assembly_2: mass 55.0475 -> 0.102452
- link right_femur_assembly: mass 55.0477 -> 0.10275
- link right_femur_assembly_2: mass 55.0477 -> 0.10275

Commit message: update urdf files

File: src/chromapi/model/urdf/robot.urdf (robot description, URDF)
Before this commit: robot chromapi, 19 links, 18 joints
Links:
- link chassis_assembly: mass 1.00501 -> 0.607607
- link left_coxa_assembly: mass 0.102452 -> 0.077795
- link left_coxa_assembly_2: mass 0.102452 -> 0.077795
- link left_femur_assembly: mass 0.10275 -> 0.077445
- link left_femur_assembly_2: mass 0.10275 -> 0.077445
- link left_tibia_assembly: mass 0.108265 -> 0.0401299
- link left_tibia_assembly_2: mass 0.108265 -> 0.0401299
- link right_coxa_assembly: mass 0.102452 -> 0.077795
- link right_coxa_assembly_2: mass 0.102452 -> 0.077795
- link right_femur_assembly: mass 0.10275 -> 0.077445
- link right_femur_assembly_2: mass 0.10275 -> 0.077445
- link right_tibia_assembly: mass 0.108265 -> 0.0401299
- link right_tibia_assembly_2: mass 0.108265 -> 0.0401299
Joints:
- joint bl_1: limit lower=-3.141592653589793 upper=3.141592653589793 effort=10 velocity=10 -> lower=-1.22173 upper=1.22173 effort=10 velocity=10; origin xyz=0.0657 0.0678 0.0355 rpy=-3.14159 0 0.785398 -> xyz=0.115884 0.0809238 0.0355 rpy=-3.14159 -0 -3.14159
- joint bl_2: limit lower=-3.141592653589793 upper=3.141592653589793 effort=10 velocity=10 -> lower=-1.5708 upper=1.74533 effort=10 velocity=10; origin xyz=0.0550631 0.034557 0.023415 rpy=-1.5708 0.785398 0.785398 -> xyz=-0.063371 0.0145 0.023415 rpy=1.5708 -1.5708 0
- joint bl_3: limit lower=-3.141592653589793 upper=3.141592653589793 effort=10 velocity=10 -> lower=-1.74533 upper=1.5708 effort=10 velocity=10; origin xyz=0.0483527 -0.0483385 0.000815 rpy=0 0 0 -> xyz=-1e-05 0.068371 0.000815 rpy=0 -0 1.5708
- joint bl_foot_frame: origin xyz=0.0303068 -0.106265 0.0152551 rpy=-2.26893 -1.57079 0.785398 -> xyz=0.0965708 -0.0537106 0.0152551 rpy=-2.26893 -1.57079 1.5708
- joint br_1: limit lower=-3.141592653589793 upper=3.141592653589793 effort=10 velocity=10 -> lower=-1.22173 upper=1.22173 effort=10 velocity=10; origin xyz=-0.0657 0.0678 0.0355 rpy=-0 0 2.35619 -> xyz=-0.0155159 0.0809238 0.0355 rpy=0 0 0
- joint br_2: limit lower=-3.141592653589793 upper=3.141592653589793 effort=10 velocity=10 -> lower=-1.5708 upper=1.74533 effort=10 velocity=10; origin xyz=0.0550631 0.034557 -0.023415 rpy=-1.5708 -0.785398 -2.35619 -> xyz=-0.063371 0.0145 -0.023415 rpy=-1.5708 -1.5708 0
- joint br_3: limit lower=-3.141592653589793 upper=3.141592653589793 effort=10 velocity=10 -> lower=-1.74533 upper=1.5708 effort=10 velocity=10; origin xyz=-0.0483385 -0.0483527 -0.000815 rpy=0 -0 -0 -> xyz=1e-05 -0.068371 -0.000815 rpy=0 0 -1.5708
- joint br_foot_frame: origin xyz=-0.106265 -0.0303068 -0.0152551 rpy=-0.872665 1.57079 -0.785398 -> xyz=0.0965708 -0.0537106 -0.0152551 rpy=-0.872665 1.57079 1.5708
- joint camera_frame: origin xyz=0.000117702 -0.0782017 0.0427998 rpy=0 -0 -1.5708 -> xyz=0.0503018 -0.065078 0.0427998 rpy=-3.14159 -1.5708 0
- joint imu_frame: origin xyz=-0.000282333 -0.000195916 0.052794 rpy=0 -0 -1.5708 -> xyz=0.0499017 0.0129279 0.052794 rpy=0 -0 -1.5708
- joint tl_1: limit lower=-3.141592653589793 upper=3.141592653589793 effort=10 velocity=10 -> lower=-1.22173 upper=1.22173 effort=10 velocity=10; origin xyz=0.0657 -0.0678 0.0355 rpy=3.14159 0 0.785398 -> xyz=0.115884 -0.0546762 0.0355 rpy=-3.14159 0 -3.14159
- joint tl_2: limit lower=-3.141592653589793 upper=3.141592653589793 effort=10 velocity=10 -> lower=-1.5708 upper=1.74533 effort=10 velocity=10; origin xyz=0.0550631 0.034557 0.023415 rpy=-1.5708 0.785398 0.785398 -> xyz=-0.063371 0.0145 0.023415 rpy=1.5708 -1.5708 0
- joint tl_3: limit lower=-3.141592653589793 upper=3.141592653589793 effort=10 velocity=10 -> lower=-1.74533 upper=1.5708 effort=10 velocity=10; origin xyz=0.0483527 -0.0483385 0.000815 rpy=0 -0 -0.785398 -> xyz=-1e-05 0.068371 0.000815 rpy=-0 -0 -3.14159
- joint tl_foot_frame: origin xyz=0.0965708 -0.0537106 0.0152551 rpy=-2.26893 -1.57079 1.5708 -> xyz=-0.0537106 -0.0965708 0.0152551 rpy=-2.26893 -1.57079 1.4e-10
- joint tr_1: limit lower=-3.141592653589793 upper=3.141592653589793 effort=10 velocity=10 -> lower=-1.22173 upper=1.22173 effort=10 velocity=10; origin xyz=-0.0657 -0.0678 0.0355 rpy=-0 0 2.35619 -> xyz=-0.0155159 -0.0546762 0.0355 rpy=-0 0 0
- joint tr_2: limit lower=-3.141592653589793 upper=3.141592653589793 effort=10 velocity=10 -> lower=-1.5708 upper=1.74533 effort=10 velocity=10; origin xyz=0.0550631 0.034557 -0.023415 rpy=-1.5708 -0.785398 -2.35619 -> xyz=-0.063371 0.0145 -0.023415 rpy=-1.5708 -1.5708 0
- joint tr_3: limit lower=-3.141592653589793 upper=3.141592653589793 effort=10 velocity=10 -> lower=-1.74533 upper=1.5708 effort=10 velocity=10; origin xyz=-0.0483385 -0.0483527 -0.000815 rpy=0 -0 -0 -> xyz=1e-05 -0.068371 -0.000815 rpy=0 0 -1.5708
- joint tr_foot_frame: origin xyz=-0.107261 -0.0303939 -0.0152551 rpy=-0.872665 1.57079 -0.785398 -> xyz=0.0973369 -0.0543534 -0.0152551 rpy=-0.872665 1.57079 1.5708

Commit message: mass fix on composite parts

File: src/chromapi/model/urdf/robot.urdf (robot description, URDF)
Before this commit: robot chromapi, 19 links, 18 joints
Links:
- link chassis_assembly: mass 0.607607 -> 0.750607; geometry collision mesh filename=package://assets/18650_li_ion_battery.stl; collision mesh filename=package://assets/18650_li_ion_battery.stl
- link left_coxa_assembly: geometry collision mesh filename=package://assets/composant2_1__corps1.stl; collision mesh filename=package://assets/composant3_1__corps1.stl
- link left_coxa_assembly_2: geometry collision mesh filename=package://assets/composant2_1__corps1.stl; collision mesh filename=package://assets/composant3_1__corps1.stl
- link left_femur_assembly: geometry collision mesh filename=package://assets/composant2_1__corps1.stl; collision mesh filename=package://assets/composant3_1__corps1.stl
- link left_femur_assembly_2: geometry collision mesh filename=package://assets/composant2_1__corps1.stl; collision mesh filename=package://assets/composant3_1__corps1.stl
- link left_tibia_assembly: mass 0.0401299 -> 0.0411317; geometry collision mesh filename=package://assets/composant2_1__corps1.stl; collision mesh filename=package://assets/composant3_1__corps1.stl
- link left_tibia_assembly_2: mass 0.0401299 -> 0.0411317; geometry collision mesh filename=package://assets/composant2_1__corps1.stl; collision mesh filename=package://assets/composant3_1__corps1.stl
- link right_coxa_assembly: geometry collision mesh filename=package://assets/composant2_1__corps1.stl; collision mesh filename=package://assets/composant3_1__corps1.stl
- link right_coxa_assembly_2: geometry collision mesh filename=package://assets/composant2_1__corps1.stl; collision mesh filename=package://assets/composant3_1__corps1.stl
- link right_femur_assembly: geometry collision mesh filename=package://assets/composant2_1__corps1.stl; collision mesh filename=package://assets/composant3_1__corps1.stl
- link right_femur_assembly_2: geometry collision mesh filename=package://assets/composant2_1__corps1.stl; collision mesh filename=package://assets/composant3_1__corps1.stl
- link right_tibia_assembly: mass 0.0401299 -> 0.0411317; geometry collision mesh filename=package://assets/composant2_1__corps1.stl; collision mesh filename=package://assets/composant3_1__corps1.stl
- link right_tibia_assembly_2: mass 0.0401299 -> 0.0411317; geometry collision mesh filename=package://assets/composant2_1__corps1.stl; collision mesh filename=package://assets/composant3_1__corps1.stl

Commit message: update robot descriptions files

File: src/chromapi/model/urdf/robot.urdf (robot description, URDF)
Before this commit: robot chromapi, 19 links, 18 joints
Joints:
- joint bl_1: origin xyz=0.115884 0.0809238 0.0355 rpy=-3.14159 -0 -3.14159 -> xyz=0.0942511 0.00365239 -0.0492694 rpy=-3.14159 -0 -3.14159
- joint bl_2: limit lower=-1.5708 upper=1.74533 effort=10 velocity=10 -> lower=-1.5708 upper=1.5708 effort=10 velocity=10
- joint bl_3: limit lower=-1.74533 upper=1.5708 effort=10 velocity=10 -> lower=-1.5708 upper=1.5708 effort=10 velocity=10
- joint br_1: origin xyz=-0.0155159 0.0809238 0.0355 rpy=0 0 0 -> xyz=-0.0371489 0.00365239 -0.0492694 rpy=0 0 0
- joint br_2: limit lower=-1.5708 upper=1.74533 effort=10 velocity=10 -> lower=-1.5708 upper=1.5708 effort=10 velocity=10
- joint br_3: limit lower=-1.74533 upper=1.5708 effort=10 velocity=10 -> lower=-1.5708 upper=1.5708 effort=10 velocity=10
- joint camera_frame: origin xyz=0.0503018 -0.065078 0.0427998 rpy=-3.14159 -1.5708 0 -> xyz=0.0286688 -0.142349 -0.0419696 rpy=-3.14159 -1.5708 0
- joint imu_frame: origin xyz=0.0499017 0.0129279 0.052794 rpy=0 -0 -1.5708 -> xyz=0.0282687 -0.0643435 -0.0319754 rpy=0 -0 -1.5708
- joint tl_1: origin xyz=0.115884 -0.0546762 0.0355 rpy=-3.14159 0 -3.14159 -> xyz=0.0942511 -0.131948 -0.0492694 rpy=-3.14159 0 -3.14159
- joint tl_2: limit lower=-1.5708 upper=1.74533 effort=10 velocity=10 -> lower=-1.5708 upper=1.5708 effort=10 velocity=10
- joint tl_3: limit lower=-1.74533 upper=1.5708 effort=10 velocity=10 -> lower=-1.5708 upper=1.5708 effort=10 velocity=10; origin xyz=-1e-05 0.068371 0.000815 rpy=-0 -0 -3.14159 -> xyz=-1e-05 0.068371 0.000815 rpy=0 0 -3.14159
- joint tl_foot_frame: origin xyz=-0.0537106 -0.0965708 0.0152551 rpy=-2.26893 -1.57079 1.4e-10 -> xyz=-0.0537106 -0.0965708 0.0152551 rpy=-2.26893 -1.57079 1.23e-10
- joint tr_1: origin xyz=-0.0155159 -0.0546762 0.0355 rpy=-0 0 0 -> xyz=-0.0371489 -0.131948 -0.0492694 rpy=-0 0 0
- joint tr_2: limit lower=-1.5708 upper=1.74533 effort=10 velocity=10 -> lower=-1.5708 upper=1.5708 effort=10 velocity=10
- joint tr_3: limit lower=-1.74533 upper=1.5708 effort=10 velocity=10 -> lower=-1.5708 upper=1.5708 effort=10 velocity=10
